File: KiCAD_PCB_Files/KiCAD_Project/Arduino_Spot_Welder.kicad_pcb (KiCad board)
At the start: 2 copper layers, 115 x 77 mm, 67 parts, among them P1 V IN, P2 MCP1407, P3 OLED_Display, P4 GND_con, P5 AutoPulse, P6 GND_con, P7 AutoPulse, Q1 MMBT3904-7-F, T1 FDB0105N407L, T2 FDB0105N407L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

Commit message: Convert to Kicad 8
Other:
- net class Default removed
